Commit message: minor

File: urdf/BMT_BRD.urdf (robot description, URDF)
Before this commit: robot Phoenix, 8 links, 7 joints
Links:
- removed link xsens_Mti30
- added link xsens; visual box size=0.05 0.05 0.05
Joints:
- joint Joint_for_ADIS: child xsens_Mti30 -> xsens

Commit message: removed yaw pitch roll joints. I think this is happening outside the base_link..

File: urdf/BMT_BRD.urdf (robot description, URDF)
Before this commit: robot Phoenix, 8 links, 7 joints
Links:
- removed link base_p
- removed link base_r
- removed link base_y
- link base_link: geometry visual cylinder length=1.5 radius=0.4
Joints:
- removed joint Joint_for_ADIS
- removed joint pitch
- removed joint roll
- removed joint yaw
- added joint Joint_for_xsens: type fixed, parent base_link, child xsens, origin xyz=0.2 0 .4 rpy=0 0 0, axis 0 0 0 
- joint Joint_for_Vectornav: parent base_r -> base_link
- joint stiff_shoulder: parent base_r -> base_link

Commit message: changed IMUs frame to xsens and turned differential on

File: urdf/BMT_BRD.urdf (robot description, URDF)
Before this commit: robot Phoenix, 5 links, 4 joints
Joints:
- joint Joint_for_xsens: origin xyz=0.2 0 .4 rpy=0 0 0 -> xyz=0 0 0 rpy=0 0 0

Commit message: added valeport launch file

File: urdf/BMT_BRD.urdf (robot description, URDF)
Before this commit: robot Phoenix, 5 links, 4 joints
Links:
- added link SVS_link; visual box size=0.05 0.05 0.05
Joints:
- added joint Joint_for_SVS: type fixed, parent base_link, child SVS_link, origin xyz=0.3 0 0.4 rpy=0 0 0, axis 0 0 0 

Commit message: added master launchfile

File: urdf/BMT_BRD.urdf (robot description, URDF)
Before this commit: robot Phoenix, 6 links, 5 joints
Links:
- added link SONAR_BMT; visual box size=0.05 0.05 0.05
- added link SONAR_UWESUB; visual box size=0.05 0.05 0.05
Joints:
- added joint JOINT_SONAR_BMT: type fixed, parent base_link, child SONAR_BMT, origin xyz=0.3 0 0.4 rpy=0 0 0, axis 0 0 0 
- added joint Joint_SONAR_UWESUB: type fixed, parent base_link, child SONAR_UWESUB, origin xyz=0.3 0 0.4 rpy=0 0 0, axis 0 0 0 

Commit message: minor

File: urdf/BMT_BRD.urdf (robot description, URDF)
Before this commit: robot Phoenix, 8 links, 7 joints
Links:
- removed link SONAR_BMT
- removed link SONAR_UWESUB
- removed link SVS_link
Joints:
- removed joint JOINT_SONAR_BMT
- removed joint Joint_SONAR_UWESUB
- removed joint Joint_for_SVS

Commit message: reintroduced the base_x,y,z,yaw,pitch,roll - they are still needed by ros_control

File: urdf/BMT_BRD.urdf (robot description, URDF)
Before this commit: robot Phoenix, 5 links, 4 joints
Links:
- added link base_pitch
- added link base_roll
- added link base_x
- added link base_y
- added link base_yaw
- added link base_z
Joints:
- added joint pitch: type continuous, parent base_yaw, child base_pitch, origin xyz=0 0 0 rpy=0 0 0, axis 0 1 0
- added joint roll: type continuous, parent base_pitch, child base_roll, origin xyz=0 0 0 rpy=0 0 0, axis 1 0 0
- added joint x: type fixed, parent base_link, child base_x, origin xyz=0 0 0 rpy=0 0 0, axis 1 0 0
- added joint y: type fixed, parent base_x, child base_y, origin xyz=0 0 0 rpy=0 0 0, axis 0 1 0
- added joint yaw: type continuous, parent base_z, child base_yaw, origin xyz=0 0 0 rpy=0 0 0, axis 0 0 1
- added joint z: type fixed, parent base_y, child base_z, origin xyz=0 0 0 rpy=0 0 0, axis 0 0 1

Commit message: bugfixes

File: urdf/BMT_BRD.urdf (robot description, URDF)
Before this commit: robot Phoenix, 11 links, 10 joints
Links:
- added link front_pitch_thruster
- added link front_yaw_thruster
- added link stern_pitch_thruster
- added link stern_yaw_thruster
- added link surge_thruster
Joints:
- added joint front_pitch_thruster_joint: type continuous, parent base_link, child front_pitch_thruster, origin xyz=1.5 0 0 rpy=0 1.571 0, axis 1 0 0
- added joint front_yaw_thruster_joint: type continuous, parent base_link, child front_yaw_thruster, origin xyz=1.6 0 0 rpy=0 0 1.571, axis 1 0 0
- added joint stern_pitch_thruster_joint: type continuous, parent base_link, child stern_pitch_thruster, origin xyz=-1.5 0 0 rpy=0 1.57 0, axis 1 0 0
- added joint stern_yaw_thruster_joint: type continuous, parent base_link, child stern_yaw_thruster, origin xyz=-1.6 0 0 rpy=0 0 1.571, axis 1 0 0
- added joint surge_thruster_joint: type continuous, parent base_link, child surge_thruster, origin xyz=-1.8 0 0 rpy=0 0 0, axis 1 0 0
- joint pitch: limit (none) -> lower=-1.39 upper=1.39 effort=50 velocity=0.147; type continuous -> revolute
- joint roll: limit (none) -> lower=-1.39 upper=1.39 effort=50 velocity=0.147
- joint x: limit (none) -> effort=30 velocity=0.3; type fixed -> continuous
- joint y: limit (none) -> effort=30 velocity=0.3; type fixed -> continuous
- joint yaw: limit (none) -> effort=50 velocity=0.147
- joint z: limit (none) -> effort=30 velocity=0.3; type fixed -> continuous

Commit message: minor

File: urdf/BMT_BRD.urdf (robot description, URDF)
Before this commit: robot Phoenix, 16 links, 15 joints
Joints:
- joint Joint_for_xsens: origin xyz=0 0 0 rpy=0 0 0 -> xyz=0 0 0 rpy=0 0 1.5707963268

Commit message: minor bugfixes

File: urdf/BMT_BRD.urdf (robot description, URDF)
Before this commit: robot Phoenix, 16 links, 15 joints
Joints:
- joint Joint_for_Vectornav: axis 0 0 0  -> (none)
- joint Joint_for_xsens: axis 0 0 0  -> (none); origin xyz=0 0 0 rpy=0 0 1.5707963268 -> xyz=0.4897 -0.08055 -0.1029 rpy=0 0 0
- joint stiff_shoulder: axis 0 0 0 -> (none)
